Commit message: Update URDF and added moveit config

File: urdf/onrobot_rg2.xacro (robot description, xacro)
@@ -28,5 +28,5 @@
         <parent link="${connected_to}"/>
         <child link="${prefix}onrobot_rg2_base_link"/>
-        <origin xyz= "0. 0. 0." rpy="0. 0. 0." />
+        <origin xyz= "0. 0. 0." rpy="0. 0. 1.57" />
       </joint>
     </xacro:unless>

File: urdf/ur3e_with_rg2.xacro (robot description, xacro)
@@ -2,4 +2,9 @@
 <robot name="ur3e_with_rg2"
   xmlns:xacro="http://wiki.ros.org/xacro">
+  <xacro:include filename="$(find ur_description)/urdf/inc/ur3e_macro.xacro"/>
+  <xacro:ur3e_robot prefix=""/>
+  <xacro:include filename="$(find wdwyl_ros1)/urdf/onrobot_rg2_model_macro.xacro" />
+  <xacro:onrobot_rg2 prefix="" connected_to="tool0"/>
+  <!-- Material definition -->
   <material name="LightGrey">
     <color rgba="0.7 0.7 0.7 1"/>
@@ -8,8 +13,10 @@
     <color rgba="0.3 0.3 0.3 1"/>
   </material>
-  <link name="world"/>
+  <material name="Mandarin">
+    <color rgba="0.9 0.5 0.1 1"/>
+  </material>
   <link name="trolley">
     <visual>
-      <origin xyz="0 0 0" rpy="0 0 0"/>
+      <origin xyz="0 0 0.45" rpy="0 0 0"/>
       <geometry>
         <box size="0.7 0.7 0.9"/>
@@ -18,13 +25,18 @@
     </visual>
     <collision>
-      <origin xyz="0 0 0" rpy="0 0 0"/>
+      <origin xyz="0 0 0.45" rpy="0 0 0"/>
       <geometry>
         <box size="0.7 0.7 0.9"/>
       </geometry>
     </collision>
+    <inertia>
+      <origin xyz="0 0 0" rpy="0 0 0"/>
+      <mass value="50"/>
+      <inertia ixx="0.1" ixy="0" ixz="0" iyy="0.1" iyz="0" izz="0.1"/>
+    </inertia>
   </link>
   <link name="task_plate">
     <visual>
-      <origin xyz="0 0 0" rpy="0 0 0"/>
+      <origin xyz="0 0 0.01" rpy="0 0 0"/>
       <geometry>
         <box size="0.495 0.32 0.02"/>
@@ -33,32 +45,39 @@
     </visual>
     <collision>
-      <origin xyz="0 0 0" rpy="0 0 0"/>
+      <origin xyz="0 0 0.01" rpy="0 0 0"/>
       <geometry>
         <box size="0.5 0.32 0.02"/>
       </geometry>
     </collision>
+    <inertia>
+      <origin xyz="0 0 0" rpy="0 0 0"/>
+      <mass value="1"/>
+      <inertia ixx="0.1" ixy="0" ixz="0" iyy="0.1" iyz="0" izz="0.1"/>
+    </inertia>
+  </link>
+  <!-- virtual End point link for planning to construct endeffector endpoint-->
+  <link name="end_point_link">
+    <visual>
+      <origin xyz="0 0 0" rpy="0 0 0"/>
+      <geometry>
+        <sphere radius="0.005"/>
+      </geometry>
+      <material name="Mandarin"/>
+    </visual>
   </link>
   <joint name="task_plate_joint" type="fixed">
     <parent link="trolley"/>
     <child link="task_plate"/>
-    <origin xyz="0 -0.1 0.45" rpy="0 0 0"/>
+    <origin xyz="0 -0.1 0.9" rpy="0 0 0"/>
   </joint>
-  <joint name="trolley_joint" type="fixed">
-    <parent link="world"/>
-    <child link="trolley"/>
-    <origin xyz="0 0 0.45" rpy="0 0 0"/>
-  </joint>
-  <joint name="fixed_base_joint" type="fixed">
+  <joint name="trolley_base_joint" type="fixed">
     <parent link="trolley"/>
     <child link="base_link"/>
-    <origin xyz="0 0.21 0.45" rpy="0 0 -3.14"/>
+    <origin xyz="0 0.21 0.9" rpy="0 0 -3.14"/>
   </joint>
-  <xacro:include filename="$(find ur_description)/urdf/inc/ur3e_macro.xacro"/>
-  <xacro:ur3e_robot prefix=""/>
-  <xacro:include filename="$(find wdwyl_ros1)/urdf/onrobot_rg2_model_macro.xacro" />
-  <xacro:onrobot_rg2 prefix="" connected_to="tool0"/>
-  <!-- <xacro:include filename="$(find realsense2_description)/urdf/_d435i.urdf.xacro"/>
-  <xacro:sensor_d435i parent="tool0" name="camera" >
-    <origin xyz="-0.0329 0 0.0732" rpy="0 -1.57 0"/>
-  </xacro:sensor_d435i> -->
+  <joint name="end_point_joint" type="fixed">
+    <parent link="tool0"/>
+    <child link="end_point_link"/>
+    <origin xyz="0 0 0.189" rpy="0 0 0"/>
+  </joint>
 </robot>

File: urdf/ur3e_with_rg2_with_trolley.urdf (robot description, URDF)
Before this commit: robot ur3e_with_rg2, 18 links, 17 joints
Links:
- added link end_point_link; visual sphere radius=0.005
- added link task_plate; collision box size=0.5 0.32 0.02; visual box size=0.495 0.32 0.02
- added link trolley; collision box size=0.7 0.7 0.9; visual box size=0.7 0.7 0.9
Joints:
- added joint end_point_joint: type fixed, parent tool0, child end_point_link, origin xyz=0 0 0.189 rpy=0 0 0
- added joint task_plate_joint: type fixed, parent trolley, child task_plate, origin xyz=0 -0.1 0.9 rpy=0 0 0
- added joint trolley_base_joint: type fixed, parent trolley, child base_link, origin xyz=0 0.21 0.9 rpy=0 0 -3.14
- joint joint0: origin xyz=0. 0. 0. rpy=0. 0. 0. -> xyz=0. 0. 0. rpy=0. 0. 1.57
