Commit message: Update urdf with base

File: urdf/ur3e_with_rg2.xacro (robot description, xacro)
@@ -1,5 +1,57 @@
 <?xml version="1.0"?>
-<robot name="ur3e_with_rg2" xmlns:xacro="http://wiki.ros.org/xacro">
-  <div id="TODO"></div>
+<robot name="ur3e_with_rg2"
+  xmlns:xacro="http://wiki.ros.org/xacro">
+  <material name="LightGrey">
+    <color rgba="0.7 0.7 0.7 1"/>
+  </material>
+  <material name="DarkGrey">
+    <color rgba="0.3 0.3 0.3 1"/>
+  </material>
+  <link name="world"/>
+  <link name="trolley">
+    <visual>
+      <origin xyz="0 0 0" rpy="0 0 0"/>
+      <geometry>
+        <box size="0.7 0.7 1"/>
+      </geometry>
+      <material name="LightGrey"/>
+    </visual>
+    <collision>
+      <origin xyz="0 0 0" rpy="0 0 0"/>
+      <geometry>
+        <box size="0.7 0.7 1"/>
+      </geometry>
+    </collision>
+  </link>
+  <link name="task_plate">
+    <visual>
+      <origin xyz="0 0 0" rpy="0 0 0"/>
+      <geometry>
+        <box size="0.495 0.32 0.02"/>
+      </geometry>
+      <material name="DarkGrey"/>
+    </visual>
+    <collision>
+      <origin xyz="0 0 0" rpy="0 0 0"/>
+      <geometry>
+        <box size="0.5 0.32 0.02"/>
+      </geometry>
+    </collision>
+  </link>
+  <joint name="task_plate_joint" type="fixed">
+    <parent link="trolley"/>
+    <child link="task_plate"/>
+    <origin xyz="0 -0.1 0.5" rpy="0 0 0"/>
+  </joint>
+  <joint name="trolley_joint" type="fixed">
+    <parent link="world"/>
+    <child link="trolley"/>
+    <origin xyz="0 0 0.5" rpy="0 0 0"/>
+  </joint>
+  <joint name="fixed_base_joint" type="fixed">
+    <parent link="trolley"/>
+    <child link="base_link"/>
+    <origin xyz="0 0.21 0.5" rpy="0 0 -3.14"/>
+  </joint>
   <xacro:include filename="$(find ur_description)/urdf/inc/ur3e_macro.xacro"/>
   <xacro:ur3e_robot prefix=""/>

Commit message: daily commit with urdf

File: urdf/ur3e_with_rg2.xacro (robot description, xacro)
@@ -13,5 +13,5 @@
       <origin xyz="0 0 0" rpy="0 0 0"/>
       <geometry>
-        <box size="0.7 0.7 1"/>
+        <box size="0.7 0.7 0.9"/>
       </geometry>
       <material name="LightGrey"/>
@@ -20,5 +20,5 @@
       <origin xyz="0 0 0" rpy="0 0 0"/>
       <geometry>
-        <box size="0.7 0.7 1"/>
+        <box size="0.7 0.7 0.9"/>
       </geometry>
     </collision>
@@ -42,15 +42,15 @@
     <parent link="trolley"/>
     <child link="task_plate"/>
-    <origin xyz="0 -0.1 0.5" rpy="0 0 0"/>
+    <origin xyz="0 -0.1 0.45" rpy="0 0 0"/>
   </joint>
   <joint name="trolley_joint" type="fixed">
     <parent link="world"/>
     <child link="trolley"/>
-    <origin xyz="0 0 0.5" rpy="0 0 0"/>
+    <origin xyz="0 0 0.45" rpy="0 0 0"/>
   </joint>
   <joint name="fixed_base_joint" type="fixed">
     <parent link="trolley"/>
     <child link="base_link"/>
-    <origin xyz="0 0.21 0.5" rpy="0 0 -3.14"/>
+    <origin xyz="0 0.21 0.45" rpy="0 0 -3.14"/>
   </joint>
   <xacro:include filename="$(find ur_description)/urdf/inc/ur3e_macro.xacro"/>
@@ -58,3 +58,7 @@
   <xacro:include filename="$(find wdwyl_ros1)/urdf/onrobot_rg2_model_macro.xacro" />
   <xacro:onrobot_rg2 prefix="" connected_to="tool0"/>
+  <!-- <xacro:include filename="$(find realsense2_description)/urdf/_d435i.urdf.xacro"/>
+  <xacro:sensor_d435i parent="tool0" name="camera" >
+    <origin xyz="-0.0329 0 0.0732" rpy="0 -1.57 0"/>
+  </xacro:sensor_d435i> -->
 </robot>

Commit message: Remove visual and collision for virtual link of endpoint

File: urdf/ur3e_with_rg2.xacro (robot description, xacro)
@@ -56,14 +56,6 @@
     </inertia>
   </link>
-  <!-- virtual End point link for planning to construct endeffector endpoint-->
-  <link name="end_point_link">
-    <visual>
-      <origin xyz="0 0 0" rpy="0 0 0"/>
-      <geometry>
-        <sphere radius="0.005"/>
-      </geometry>
-      <material name="Mandarin"/>
-    </visual>
-  </link>
+  <!-- virtual End point link for planning to construct endeffector endpoint, thus, no visual or collision aspect -->
+  <link name="end_point_link"/>
   <joint name="task_plate_joint" type="fixed">
     <parent link="trolley"/>
@@ -79,5 +71,5 @@
     <parent link="tool0"/>
     <child link="end_point_link"/>
-    <origin xyz="0 0 0.189" rpy="0 0 0"/>
+    <origin xyz="0 0 0.20" rpy="0 0 0"/>
   </joint>
 </robot>

File: urdf/ur3e_with_rg2_with_trolley.urdf (robot description, URDF)
Before this commit: robot ur3e_with_rg2, 21 links, 20 joints
Links:
- link end_point_link: geometry 
Joints:
- joint end_point_joint: origin xyz=0 0 0.189 rpy=0 0 0 -> xyz=0 0 0.20 rpy=0 0 0

Commit message: Update launch file change

File: urdf/ur3e_with_rg2.xacro (robot description, xacro)
@@ -2,8 +2,4 @@
 <robot name="ur3e_with_rg2"
   xmlns:xacro="http://wiki.ros.org/xacro">
-  <xacro:include filename="$(find ur_description)/urdf/inc/ur3e_macro.xacro"/>
-  <xacro:ur3e_robot prefix=""/>
-  <xacro:include filename="$(find wdwyl_ros1)/urdf/onrobot_rg2_model_macro.xacro" />
-  <xacro:onrobot_rg2 prefix="" connected_to="tool0"/>
   <!-- Material definition -->
   <material name="LightGrey">
@@ -12,7 +8,4 @@
   <material name="DarkGrey">
     <color rgba="0.3 0.3 0.3 1"/>
-  </material>
-  <material name="Mandarin">
-    <color rgba="0.9 0.5 0.1 1"/>
   </material>
   <link name="trolley">
@@ -58,4 +51,8 @@
   <!-- virtual End point link for planning to construct endeffector endpoint, thus, no visual or collision aspect -->
   <link name="end_point_link"/>
+  <xacro:include filename="$(find ur_description)/urdf/inc/ur3e_macro.xacro"/>
+  <xacro:ur3e_robot prefix=""/>
+  <xacro:include filename="$(find wdwyl_ros1)/urdf/onrobot_rg2_model_macro.xacro" />
+  <xacro:onrobot_rg2 prefix="" connected_to="tool0"/>
   <joint name="task_plate_joint" type="fixed">
     <parent link="trolley"/>
