Commit message: added classification integration

File: manipulation/urdf/ur3e_with_rg2.xacro (robot description, xacro)
@@ -13,5 +13,5 @@
       <origin xyz="0 0 0.45" rpy="0 0 0"/>
       <geometry>
-        <box size="0.7 0.7 0.9"/>
+        <box size="0.73 0.71 0.9"/>
       </geometry>
       <material name="LightGrey"/>
@@ -20,5 +20,5 @@
       <origin xyz="0 0 0.45" rpy="0 0 0"/>
       <geometry>
-        <box size="0.7 0.7 0.9"/>
+        <box size="0.73 0.71 0.9"/>
       </geometry>
     </collision>

File: manipulation/urdf/ur3e_with_rg2_with_trolley.urdf (robot description, URDF)
Before this commit: robot ur3e_with_rg2, 21 links, 20 joints
Links:
- link trolley: geometry collision box size=2.73 0.71 0.9; visual box size=2.73 0.71 0.9
